File: STM32_V1.kicad_pcb (KiCad board)
At the start: 4 copper layers, 1 part, among them U1 AD6644

Commit message: updated 5530
Parts:
- added U2: STM32F411CEUx, Package_DFN_QFN:QFN-48-1EP_7x7mm_P0.5mm_EP5.6x5.6mm, F.Cu at (155.0, 84.5)
- added U3: MPU-6050, Sensor_Motion:InvenSense_QFN-24_4x4mm_P0.5mm, F.Cu at (121.8, 90.0)
- U1: value AD6644 -> AMS1117-3.3; footprint Package_QFP:TQFP-52-1EP_10x10mm_P0.65mm_EP6.5x6.5mm -> Package_TO_SOT_SMD:SOT-223-3_TabPin2
- moved U1 17.9 mm to (132.6, 81.2)
Connections:
- U1 pad 1: Net-(U1-Pad1) -> unconnected-(U1-Pad1)
- U1 pad 2: Net-(U1-Pad10) -> unconnected-(U1-Pad2)
Routing:
- net input: track 10.3 -> 0.00 mm
- net Net-(U1-Pad10): track 6.75 -> 0.00 mm, vias 2 -> 0
