File: STM32_V1.kicad_sch (KiCad schematic)
At the start: 3 parts

Commit message: updated 5530
Parts:
- gave numbers to parts that had none: 3
Changed lines of the file:
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@@
   (symbol (lib_id "Regulator_Linear:AMS1117-3.3") (at 93.726 219.202 0) (unit 1)
     (in_bom yes) (on_board yes) (fields_autoplaced)
-    (property "Reference" "U?" (id 0) (at 93.726 212.09 0))
+    (property "Reference" "U1" (id 0) (at 93.726 212.09 0))
     (property "Value" "AMS1117-3.3" (id 1) (at 93.726 214.63 0))
     (property "Footprint" "Package_TO_SOT_SMD:SOT-223-3_TabPin2" (id 2) (at 93.726 214.122 0)
@@
     (pin "3")
   )
+  (symbol (lib_id "power:GND") (at 200.66 94.996 0) (unit 1)
+    (in_bom yes) (on_board yes)
+    (property "Reference" "#PWR?" (id 0) (at 200.66 101.346 0)
+      (effects (font (size 1.27 1.27)) hide)
+    )
+    (property "Value" "GND" (id 1) (at 206.502 98.044 0)
+      (effects (font (size 1.27 1.27)) hide)
+    )
+    (property "Footprint" "" (id 2) (at 200.66 94.996 0)
+      (effects (font (size 1.27 1.27)) hide)
+    )
+    (property "Datasheet" "" (id 3) (at 200.66 94.996 0)
+      (effects (font (size 1.27 1.27)) hide)
+    )
+    (pin "1")
+  )
   (symbol (lib_id "Sensor_Motion:MPU-6050") (at 333.502 173.228 0) (unit 1)
     (in_bom yes) (on_board yes) (fields_autoplaced)
-    (property "Reference" "U?" (id 0) (at 335.5214 190.246 0)
+    (property "Reference" "U3" (id 0) (at 335.5214 190.246 0)
       (effects (font (size 1.27 1.27)) (justify left))
     )
@@
     (pin "9")
   )
+  (symbol (lib_id "power:+3.3V") (at 228.092 66.294 0) (unit 1)
+    (in_bom yes) (on_board yes)
+    (property "Reference" "#PWR?" (id 0) (at 228.092 70.104 0)
+      (effects (font (size 1.27 1.27)) hide)
+    )
+    (property "Value" "+3.3V" (id 1) (at 228.092 62.738 0))
+    (property "Footprint" "" (id 2) (at 228.092 66.294 0)
+      (effects (font (size 1.27 1.27)) hide)
+    )
+    (property "Datasheet" "" (id 3) (at 228.092 66.294 0)
+      (effects (font (size 1.27 1.27)) hide)
+    )
+    (pin "1")
+  )
   (symbol (lib_id "MCU_ST_STM32F4:STM32F411CEUx") (at 177.546 102.108 0) (unit 1)
     (in_bom yes) (on_board yes)
-    (property "Reference" "U?" (id 0) (at 169.926 62.23 0)
+    (property "Reference" "U2" (id 0) (at 169.926 62.23 0)
       (effects (font (size 1.27 1.27)) (justify left))
     )
@@
   )
   (symbol_instances
+    (path "/822ba726-1168-4fe4-84db-5162ce850b90"
+      (reference "#PWR?") (unit 1) (value "GND") (footprint "")
+    )
+    (path "/c0810860-6483-467b-b1d9-d9b6bcda5b31"
+      (reference "#PWR?") (unit 1) (value "+3.3V") (footprint "")
+    )
     (path "/7072e856-6e20-459b-83ca-f3d073fff20b"
-      (reference "U?") (unit 1) (value "AMS1117-3.3") (footprint "Package_TO_SOT_SMD:SOT-223-3_TabPin2")
+      (reference "U1") (unit 1) (value "AMS1117-3.3") (footprint "Package_TO_SOT_SMD:SOT-223-3_TabPin2")
+    )
+    (path "/f002c4d3-baf8-41c6-8910-e41156cb5309"
+      (reference "U2") (unit 1) (value "STM32F411CEUx") (footprint "Package_DFN_QFN:QFN-48-1EP_7x7mm_P0.5mm_EP5.6x5.6mm")
     )
     (path "/9615ef73-ed5b-4903-b913-7103211fa661"
-      (reference "U?") (unit 1) (value "MPU-6050") (footprint "Sensor_Motion:InvenSense_QFN-24_4x4mm_P0.5mm")
-    )
-    (path "/f002c4d3-baf8-41c6-8910-e41156cb5309"
-      (reference "U?") (unit 1) (value "STM32F411CEUx") (footprint "Package_DFN_QFN:QFN-48-1EP_7x7mm_P0.5mm_EP5.6x5.6mm")
+      (reference "U3") (unit 1) (value "MPU-6050") (footprint "Sensor_Motion:InvenSense_QFN-24_4x4mm_P0.5mm")
     )
   )
